Commit message: Clean Newton teleop examples and assets

File: isaaclab_arena/assets/robots/abb/irb1200_7_70/irb1200_7_70.urdf (robot description, URDF)
Before this commit: robot abb_irb1200_7_70, 10 links, 9 joints
Links:
- link base_link: geometry collision mesh filename=/workspaces/isaaclab_arena/isaaclab_arena/assets/robots/abb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; visual mesh filename=/workspaces/isaaclab_arena/isaaclab_arena/assets/robots/abb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
- link link_1: geometry collision mesh filename=/workspaces/isaaclab_arena/isaaclab_arena/assets/robots/abb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; visual mesh filename=/workspaces/isaaclab_arena/isaaclab_arena/assets/robots/abb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
- link link_2: geometry collision mesh filename=/workspaces/isaaclab_arena/isaaclab_arena/assets/robots/abb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; visual mesh filename=/workspaces/isaaclab_arena/isaaclab_arena/assets/robots/abb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
- link link_3: geometry collision mesh filename=/workspaces/isaaclab_arena/isaaclab_arena/assets/robots/abb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; visual mesh filename=/workspaces/isaaclab_arena/isaaclab_arena/assets/robots/abb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
- link link_4: geometry collision mesh filename=/workspaces/isaaclab_arena/isaaclab_arena/assets/robots/abb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; visual mesh filename=/workspaces/isaaclab_arena/isaaclab_arena/assets/robots/abb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
- link link_5: geometry collision mesh filename=/workspaces/isaaclab_arena/isaaclab_arena/assets/robots/abb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; visual mesh filename=/workspaces/isaaclab_arena/isaaclab_arena/assets/robots/abb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
- link link_6: geometry collision mesh filename=/workspaces/isaaclab_arena/isaaclab_arena/assets/robots/abb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; visual mesh filename=/workspaces/isaaclab_arena/isaaclab_arena/assets/robots/abb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
